File: Aquila_mobile.brd (EAGLE design)
At the start: 92.2 x 64.3 mm, 177 parts, among them J200 DNI, J201 DNI, J210 DNI, J220 DNI, J300 78646-3001, J310 U.FL_CONNECTOR, J400 10103593, K100 1376408-1_DDR1_1.8V_REDUCED, Q300 DTC143ZET1G, Q301 DTC143ZET1G, U300 QUECTEL_M10_R, U410 BQ24032ARHLR, U420 TPS63002DRC, U430 TPS7A7001

Commit message: Layout: fix errata into U410 and U420 pads
Pads from U410 and U420 designators didn't contain solder mask (tStop)
and stencil mask (tCream). This patch corrects designs files and gerbers.

Signed-off-by: Pau Pajuelo <ppajuel@gmail.com>
Parts:
- U410: device texas-MOD:QFN20_3,5X4,5 -> ppajuel_library:BQ24032ARHLR
Connections:
- net DGND: now also U410.21; no longer U410.EXP, U410.EXP@1, U410.EXP@10, U410.EXP@11, U410.EXP@12, U410.EXP@2, U410.EXP@3, U410.EXP@4, U410.EXP@5, U410.EXP@6, U410.EXP@7, U410.EXP@8, U410.EXP@9
Changed lines of the file:
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@@
 <layer number="27" name="tValues" color="7" fill="1" visible="no" active="yes"/>
 <layer number="28" name="bValues" color="7" fill="1" visible="no" active="yes"/>
-<layer number="29" name="tStop" color="7" fill="3" visible="no" active="yes"/>
+<layer number="29" name="tStop" color="7" fill="3" visible="yes" active="yes"/>
 <layer number="30" name="bStop" color="7" fill="6" visible="no" active="yes"/>
 <layer number="31" name="tCream" color="7" fill="4" visible="no" active="yes"/>
@@
 <attribute name="VALUE" x="79.9654" y="12.6732" size="1.27" layer="27"/>
 </element>
-<element name="U410" library="texas-MOD" package="QFN20_3,5X4,5" value="BQ24032ARHLR" x="63.0682" y="34.1122" smashed="yes" rot="R180">
+<element name="U410" library="ppajuel_library" package="BQ24032ARHLR" value="BQ24032ARHLR" x="63.0682" y="34.1122" smashed="yes" rot="R180">
 <attribute name="NAME" x="58.4962" y="32.4358" size="0.6096" layer="25"/>
 <attribute name="VALUE" x="59.2582" y="37.6682" size="1.27" layer="27" rot="R180"/>
@@
 <contactref element="R414" pad="1"/>
 <contactref element="U410" pad="11"/>
-<contactref element="U410" pad="EXP"/>
+<contactref element="U410" pad="21"/>
 <contactref element="U420" pad="3"/>
 <contactref element="U420" pad="9"/>
@@
 <wire x1="54.7878" y1="7.2898" x2="54.7878" y2="4.3942" width="0.2032" layer="16"/>
 <wire x1="54.7878" y1="4.3942" x2="54.991" y2="4.191" width="0.2032" layer="16"/>
-<contactref element="U410" pad="EXP@1"/>
-<contactref element="U410" pad="EXP@7"/>
-<contactref element="U410" pad="EXP@8"/>
-<contactref element="U410" pad="EXP@9"/>
-<contactref element="U410" pad="EXP@10"/>
-<contactref element="U410" pad="EXP@11"/>
-<contactref element="U410" pad="EXP@12"/>
-<contactref element="U410" pad="EXP@2"/>
-<contactref element="U410" pad="EXP@3"/>
-<contactref element="U410" pad="EXP@4"/>
-<contactref element="U410" pad="EXP@5"/>
-<contactref element="U410" pad="EXP@6"/>
 <contactref element="U420" pad="EXP@1"/>
 <contactref element="U420" pad="EXP@2"/>
@@
 <wire x1="57.8866" y1="34.1884" x2="62.5856" y2="34.1884" width="0.508" layer="1"/>
 <wire x1="62.5856" y1="34.1884" x2="63.0682" y2="34.671" width="0.508" layer="1"/>
-<wire x1="59.8432" y1="33.3622" x2="57.8104" y2="33.3622" width="0.508" layer="1"/>
+<wire x1="59.8182" y1="33.3622" x2="57.8104" y2="33.3622" width="0.508" layer="1"/>
 <wire x1="57.8104" y1="33.3622" x2="57.646" y2="33.3622" width="0.508" layer="1"/>
 <wire x1="57.646" y1="33.3622" x2="57.5818" y2="33.4264" width="0.508" layer="1"/>
@@
 <contactref element="K100" pad="126"/>
 <wire x1="51.5544" y1="22.9866" x2="51.5544" y2="20.2778" width="0.2032" layer="1"/>
-<wire x1="64.3182" y1="31.3872" x2="64.3182" y2="29.7888" width="0.2032" layer="1"/>
+<wire x1="64.3182" y1="31.3622" x2="64.3182" y2="29.7888" width="0.2032" layer="1"/>
 <wire x1="64.3182" y1="29.7888" x2="64.516" y2="29.591" width="0.2032" layer="1"/>
 <wire x1="64.516" y1="29.591" x2="65.532" y2="29.591" width="0.2032" layer="1"/>
@@
 <wire x1="66.0146" y1="35.6616" x2="66.0146" y2="35.7242" width="0.2032" layer="1"/>
 <wire x1="66.0146" y1="35.7242" x2="66.9172" y2="36.6268" width="0.2032" layer="1"/>
-<wire x1="64.8182" y1="36.8372" x2="66.7068" y2="36.8372" width="0.2032" layer="1"/>
+<wire x1="64.8182" y1="36.8622" x2="66.7068" y2="36.8372" width="0.2032" layer="1"/>
 <wire x1="66.7068" y1="36.8372" x2="66.9172" y2="36.6268" width="0.2032" layer="1"/>
 <wire x1="54.8386" y1="25.3238" x2="55.8038" y2="25.3238" width="0.2032" layer="1"/>
@@
 <wire x1="64.516" y1="38.6588" x2="64.3128" y2="38.4556" width="0.2032" layer="1"/>
 <wire x1="64.3128" y1="38.4556" x2="64.3128" y2="36.8426" width="0.2032" layer="1"/>
-<wire x1="64.3128" y1="36.8426" x2="64.3182" y2="36.8372" width="0.2032" layer="1"/>
+<wire x1="64.3128" y1="36.8426" x2="64.3182" y2="36.8622" width="0.2032" layer="1"/>
 <wire x1="52.217" y1="23.0378" x2="52.217" y2="23.2864" width="0.2032" layer="1"/>
 <wire x1="52.217" y1="23.2864" x2="52.6542" y2="23.7236" width="0.2032" layer="1"/>
@@
 <wire x1="63.8182" y1="38.7484" x2="63.8182" y2="38.4182" width="0.4064" layer="1"/>
 <wire x1="63.8182" y1="38.4182" x2="63.8048" y2="38.4048" width="0.4064" layer="1"/>
-<wire x1="63.8182" y1="36.8372" x2="63.8182" y2="38.3914" width="0.3048" layer="1"/>
+<wire x1="63.8182" y1="36.8622" x2="63.8182" y2="38.3914" width="0.3048" layer="1"/>
 <wire x1="63.8182" y1="38.3914" x2="63.8048" y2="38.4048" width="0.3048" layer="1"/>
 <wire x1="63.0056" y1="42.6076" x2="62.7634" y2="42.8498" width="0.2032" layer="1"/>
@@
 <wire x1="60.579" y1="39.5986" x2="61.341" y2="38.8366" width="0.2032" layer="1"/>
 <wire x1="61.341" y1="38.8366" x2="61.341" y2="36.86" width="0.2032" layer="1"/>
-<wire x1="61.341" y1="36.86" x2="61.3182" y2="36.8372" width="0.2032" layer="1"/>
+<wire x1="61.341" y1="36.86" x2="61.3182" y2="36.8622" width="0.2032" layer="1"/>
 <wire x1="60.579" y1="39.5986" x2="60.579" y2="40.8822" width="0.2032" layer="1"/>
 <wire x1="60.579" y1="40.8822" x2="60.5536" y2="40.9076" width="0.2032" layer="1"/>
@@
 <wire x1="62.5856" y1="39.7256" x2="61.8236" y2="38.9636" width="0.2032" layer="1"/>
 <wire x1="61.8236" y1="38.9636" x2="61.8236" y2="36.8426" width="0.2032" layer="1"/>
-<wire x1="61.8236" y1="36.8426" x2="61.8182" y2="36.8372" width="0.2032" layer="1"/>
+<wire x1="61.8236" y1="36.8426" x2="61.8182" y2="36.8622" width="0.2032" layer="1"/>
 </signal>
 <signal name="N$9">
@@
 <contactref element="U410" pad="10"/>
 <wire x1="59.3208" y1="36.6268" x2="59.3208" y2="35.3846" width="0.2032" layer="1"/>
-<wire x1="59.3208" y1="35.3846" x2="59.8432" y2="34.8622" width="0.2032" layer="1"/>
+<wire x1="59.3208" y1="35.3846" x2="59.8182" y2="34.8622" width="0.2032" layer="1"/>
 </signal>
 <signal name="N$10">
 <contactref element="R414" pad="2"/>
 <contactref element="U410" pad="13"/>
-<wire x1="61.8182" y1="31.3872" x2="61.8182" y2="29.2418" width="0.2032" layer="1"/>
+<wire x1="61.8182" y1="31.3622" x2="61.8182" y2="29.2418" width="0.2032" layer="1"/>
 <wire x1="61.8182" y1="29.2418" x2="61.1632" y2="28.5868" width="0.2032" layer="1"/>
 </signal>
@@
 <contactref element="R415" pad="2"/>
 <contactref element="U410" pad="14"/>
-<wire x1="62.3182" y1="31.3872" x2="62.3182" y2="29.4638" width="0.2032" layer="1"/>
+<wire x1="62.3182" y1="31.3622" x2="62.3182" y2="29.4638" width="0.2032" layer="1"/>
 <wire x1="62.3182" y1="29.4638" x2="63.1952" y2="28.5868" width="0.2032" layer="1"/>
 </signal>
@@
 <wire x1="64.6176" y1="40.9076" x2="64.555" y2="40.9076" width="0.2032" layer="1"/>
 <wire x1="62.3316" y1="38.6842" x2="62.3316" y2="36.8506" width="0.2032" layer="1"/>
-<wire x1="62.3316" y1="36.8506" x2="62.3182" y2="36.8372" width="0.2032" layer="1"/>
+<wire x1="62.3316" y1="36.8506" x2="62.3182" y2="36.8622" width="0.2032" layer="1"/>
 <wire x1="62.3316" y1="38.6842" x2="62.3316" y2="38.862" width="0.2032" layer="1"/>
 <wire x1="62.3316" y1="38.862" x2="62.3316" y2="38.8874" width="0.2032" layer="1"/>
@@
 <wire x1="88.9" y1="14.986" x2="88.9078" y2="14.9782" width="0.4064" layer="1"/>
 <wire x1="89.4588" y1="14.4702" x2="89.4666" y2="14.478" width="0.4064" layer="1"/>
-<wire x1="63.3182" y1="31.3872" x2="63.3182" y2="30.0442" width="1.016" layer="1"/>
+<wire x1="63.3182" y1="31.3622" x2="63.3182" y2="30.0442" width="1.016" layer="1"/>
 <wire x1="63.3182" y1="30.0442" x2="63.2968" y2="30.0228" width="1.016" layer="1"/>
-<wire x1="62.8182" y1="31.3872" x2="63.3182" y2="31.3872" width="0.2032" layer="1"/>
-<wire x1="63.3182" y1="31.3872" x2="63.8182" y2="31.3872" width="0.2032" layer="1"/>
+<wire x1="62.8182" y1="31.3622" x2="63.3182" y2="31.3622" width="0.2032" layer="1"/>
+<wire x1="63.3182" y1="31.3622" x2="63.8182" y2="31.3622" width="0.2032" layer="1"/>
 <wire x1="65.2272" y1="28.5868" x2="64.8344" y2="28.5868" width="0.4572" layer="1"/>
 <wire x1="64.8344" y1="28.5868" x2="63.7286" y2="29.6926" width="0.4572" layer="1"/>
@@
 <wire x1="65.278" y1="39.8018" x2="63.9826" y2="39.8018" width="0.4064" layer="1"/>
 <wire x1="63.9826" y1="39.8018" x2="63.5762" y2="39.3954" width="0.4064" layer="1"/>
-<wire x1="63.3182" y1="36.8372" x2="62.8182" y2="36.8372" width="0.2032" layer="1"/>
+<wire x1="63.3182" y1="36.8622" x2="62.8182" y2="36.8622" width="0.2032" layer="1"/>
 <via x="88.4428" y="20.4724" extent="1-16" drill="0.6" diameter="0.127"/>
 <via x="67.4624" y="44.6024" extent="1-16" drill="0.6" diameter="0.127"/>
@@
 <wire x1="63.5762" y1="39.3954" x2="63.0682" y2="38.8874" width="0.4064" layer="1"/>
 <wire x1="63.0682" y1="38.8874" x2="63.0682" y2="37.3888" width="0.4064" layer="1"/>
-<wire x1="62.8182" y1="36.8372" x2="63.05" y2="36.8372" width="0.2032" layer="1"/>
+<wire x1="62.8182" y1="36.8622" x2="63.05" y2="36.8372" width="0.2032" layer="1"/>
 <wire x1="63.05" y1="36.8372" x2="63.0682" y2="36.8554" width="0.2032" layer="1"/>
 <wire x1="63.0682" y1="36.8554" x2="63.0682" y2="37.3888" width="0.4064" layer="1"/>
@@
 <wire x1="66.3956" y1="30.8356" x2="66.9798" y2="31.4198" width="0.3048" layer="1"/>
 <wire x1="66.3956" y1="30.8356" x2="59.9948" y2="30.8356" width="0.3048" layer="16"/>
-<wire x1="61.3182" y1="31.3872" x2="60.5464" y2="31.3872" width="0.3048" layer="1"/>
+<wire x1="61.3182" y1="31.3622" x2="60.5464" y2="31.3872" width="0.3048" layer="1"/>
 <wire x1="60.5464" y1="31.3872" x2="59.9948" y2="30.8356" width="0.3048" layer="1"/>
 </signal>
